File: pcb/banc d'essais l_h.kicad_pcb (KiCad board)
At the start: 2 copper layers, 2 parts

Commit message: création des pond du pcb
Routing:
- net Net-(A1-D4): track 67.3 -> 37.2 mm, vias 0 -> 4
- net Led test +: track 38.8 -> 59.7 mm, vias 0 -> 6
- net Net-(A1-D12): track 34.4 -> 49.5 mm, vias 0 -> 2
- net Net-(A1-D2): track 78.8 -> 65.7 mm, vias 0 -> 2
- net Led test -: track 38.5 -> 45.6 mm, vias 0 -> 2
- net Net-(A1-D11): track 36.5 -> 30.2 mm
- net Net-(A1-D5): track 33.0 -> 35.9 mm
- net Net-(A1-D3): track 36.0 -> 37.2 mm
